Commit message: updated planning algorithms, updated Cmakefiles to prevent message and service compiling errors, added gitignore files

File: espeleo_planner/urdf/espeleo2_low_poly.urdf (robot description, URDF)
Before this commit: robot espeleo, 13 links, 12 joints
Links:
- removed link d435i_link
- removed link imu_link
- removed link only_visual_t265
- removed link os1_sensor
- removed link sensor_tower
- link chassis: geometry collision box size=0.54 0.27 0.145; visual mesh filename=package://espeleo_planner/espeleo_planner/urdf/stl/corpo.stl scale=0.001 0.001 0.001
- link left_back_wheel: geometry collision cylinder length=0.043 radius=0.14; visual mesh filename=package://espeleo_planner/espeleo_planner/urdf/stl/roda_esq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 scale=0.001 0.001 0.001
- link left_front_wheel: geometry collision cylinder length=0.043 radius=0.14; visual mesh filename=package://espeleo_planner/espeleo_planner/urdf/stl/roda_esq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 scale=0.001 0.001 0.001
- link left_middle_wheel: geometry collision cylinder length=0.043 radius=0.14; visual mesh filename=package://espeleo_planner/espeleo_planner/urdf/stl/roda_esq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 scale=0.001 0.001 0.001
- link right_back_wheel: geometry collision cylinder length=0.043 radius=0.14; visual mesh filename=package://espeleo_planner/espeleo_planner/urdf/stl/roda_esq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 scale=0.001 0.001 0.001
- link right_front_wheel: geometry collision cylinder length=0.043 radius=0.14; visual mesh filename=package://espeleo_planner/espeleo_planner/urdf/stl/roda_esq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 scale=0.001 0.001 0.001
- link right_middle_wheel: geometry collision cylinder length=0.043 radius=0.14; visual mesh filename=package://espeleo_planner/espeleo_planner/urdf/stl/roda_esq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 scale=0.001 0.001 0.001
Joints:
- removed joint imu_joint
- removed joint laser_joint
- removed joint realsense_d435_joint
- removed joint realsense_t265_joint
- removed joint sensor_tower_joint

File: espeleo_planner/urdf/espeleo2_low_poly_prismatic.urdf (robot description, URDF)
Before this commit: robot espeleo, 10 links, 9 joints
Links:
- link z_prismatic: mass 0.01 -> 1.0
Joints:
- joint z_to_world: axis 0 1 0 -> 0 0 1
